File: Hardware/GBDump/GBDump.kicad_pcb (KiCad board)
At the start: 2 copper layers, 136.8 x 55.9 mm, 19 parts, among them J1 Conn_01x06, J2 Micro_SD_Card_Det_Hirose_DM3AT, J3 Conn_01x06, U2 TXB0108PW, U3 TXB0108PW, U4 TXB0108PW, U5 Cartridge_Bus, U6 TXB0108PW

Commit message: Finished silkscreen, generated gerbers.
Other:
- rule pad_to_mask_clearance: 0 -> 0.0508
- board text added: "3.3V"
- board text added: "5V"
- board text added: "Cubby DeBry"
- board text added: "GND"
- board text added: "MISO"
- board text added: "MOSI"
- board text added: "NSS"
- board text added: "SCK"
- board text added: "SPI1"
- board text added: "SPI2"
- board text added: "U of U Embedded Systems 2025"
- board text added: "V Select"
